File: KiCAD/MicroController.sch (KiCad schematic (older format))
At the start: 23 parts, among them J2 Conn_02x03_Odd_Even, SW1 SW_DPST_x2, U3 ATMEGA2560-16AU, Y1 16MHz

Commit message: transfer for mechanical step
Parts:
- removed SW1: SW_DPST_x2, Buttons_Switches_SMD:SW_SPST_B3U-1000P, symbol SW_DPST_x2
- added R28: 10k, Resistors_SMD:R_0805, symbol R
- added SW1, SW2: SW_SPST, Buttons_Switches_SMD:SW_SPST_B3U-1000P, symbol SW_SPST
- L2: footprint (none) -> kicad-footprints:L-1008; Part MH2029-300Y -> https://www.digikey.ca/product-detail/en/wurth-electronics-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
- MK2, MK3, MK4: footprint (none) -> Mounting_Holes:MountingHole_3.2mm_M3
- Y1: footprint (none) -> Crystals:Crystal_HC49-U_Vertical
Connections:
- net MISO is gone; now on net 50(MISO): J2.1 (Pin_1)
- net MOSI is gone; now on net 51(MOSI): J2.4 (Pin_4)
- net SCK is gone; now on net 52(SCK): J2.3 (Pin_3)
- net +5V: now also R28.2
- net 34: now also D6.2 (A)
- net 35: now also D5.2 (A)
- net 36: now also D4.2 (A)
- net 37: now also SW2.1 (A)
- net GND: now also SW1.2 (B), SW2.2 (B)
- net RESET: now also R28.1, SW1.1 (A)
Other:
- moved on the sheet: MK4
Changed lines of the file:
@@
 $EndComp
 $Comp
-L GND #PWR018
+L GND #PWR21
 U 1 1 5A91BF4A
 P 3350 7550
-F 0 "#PWR018" H 3350 7300 50  0001 C CNN
+F 0 "#PWR21" H 3350 7300 50  0001 C CNN
 F 1 "GND" H 3350 7400 50  0000 C CNN
 F 2 "" H 3350 7550 50  0001 C CNN
@@
 $EndComp
 $Comp
-L +5V #PWR019
+L +5V #PWR20
 U 1 1 5A91C010
 P 3100 1050
-F 0 "#PWR019" H 3100 900 50  0001 C CNN
+F 0 "#PWR20" H 3100 900 50  0001 C CNN
 F 1 "+5V" H 3100 1190 50  0000 C CNN
 F 2 "" H 3100 1050 50  0001 C CNN
@@
 $EndComp
 $Comp
-L +5V #PWR020
+L +5V #PWR25
 U 1 1 5A91C19A
 P 7400 950
-F 0 "#PWR020" H 7400 800 50  0001 C CNN
+F 0 "#PWR25" H 7400 800 50  0001 C CNN
 F 1 "+5V" H 7400 1090 50  0000 C CNN
 F 2 "" H 7400 950 50  0001 C CNN
@@
 $EndComp
 $Comp
-L GND #PWR021
+L GND #PWR26
 U 1 1 5AA06A82
 P 7400 1700
-F 0 "#PWR021" H 7400 1450 50  0001 C CNN
+F 0 "#PWR26" H 7400 1450 50  0001 C CNN
 F 1 "GND" H 7400 1550 50  0000 C CNN
 F 2 "" H 7400 1700 50  0001 C CNN
@@
 F 0 "Y1" H 850 2750 50  0000 C CNN
 F 1 "16MHz" H 850 2450 50  0000 C CNN
-F 2 "" H 850 2600 50  0001 C CNN
-F 3 "" H 850 2600 50  0001 C CNN
+F 2 "Crystals:Crystal_HC49-U_Vertical" H 850 2600 50  0001 C CNN
+F 3 "https://www.digikey.ca/products/en?keywords=X433-ND%20" H 850 2600 50  0001 C CNN
 	1    850  2600
 	-1   0    0    1
@@
 $EndComp
 $Comp
-L GND #PWR022
+L GND #PWR19
 U 1 1 5AA0A088
 P 850 3050
-F 0 "#PWR022" H 850 2800 50  0001 C CNN
+F 0 "#PWR19" H 850 2800 50  0001 C CNN
 F 1 "GND" H 850 2900 50  0000 C CNN
 F 2 "" H 850 3050 50  0001 C CNN
@@
 Connection ~ 850  3000
 $Comp
-L +5V #PWR023
+L +5V #PWR23
 U 1 1 5AA0ACDC
 P 4150 1050
-F 0 "#PWR023" H 4150 900 50  0001 C CNN
+F 0 "#PWR23" H 4150 900 50  0001 C CNN
 F 1 "+5V" H 4150 1190 50  0000 C CNN
 F 2 "" H 4150 1050 50  0001 C CNN
@@
 F 0 "L2" V 3850 1150 50  0000 C CNN
 F 1 "10uH" V 3975 1150 50  0000 C CNN
-F 2 "" H 3900 1150 50  0001 C CNN
+F 2 "kicad-footprints:L-1008" H 3900 1150 50  0001 C CNN
 F 3 "" H 3900 1150 50  0001 C CNN
-F 4 "MH2029-300Y" V 3900 1150 60  0001 C CNN "Part"
+F 4 "https://www.digikey.ca/product-detail/en/wurth-electronics-inc/74479887310A/732-4516-1-ND/4120134" V 3900 1150 60  0001 C CNN "Part"
 	1    3900 1150
 	0    1    1    0
@@
 $EndComp
 $Comp
-L GND #PWR024
+L GND #PWR22
 U 1 1 5AA0B0AB
 P 3600 1450
-F 0 "#PWR024" H 3600 1200 50  0001 C CNN
+F 0 "#PWR22" H 3600 1200 50  0001 C CNN
 F 1 "GND" H 3600 1300 50  0000 C CNN
 F 2 "" H 3600 1450 50  0001 C CNN
@@
 Wire Wire Line
 	10150 1450 10450 1450
-Text GLabel 9500 1250 0    49   Input ~ 0
-MISO
-Text GLabel 9500 1350 0    49   Input ~ 0
-SCK
 Text GLabel 9500 1450 0    49   Input ~ 0
 RESET
-Text GLabel 10300 1350 2    49   Input ~ 0
-MOSI
-$Comp
-L +5V #PWR025
+$Comp
+L +5V #PWR29
 U 1 1 5AA0C848
 P 10450 1100
-F 0 "#PWR025" H 10450 950 50  0001 C CNN
+F 0 "#PWR29" H 10450 950 50  0001 C CNN
 F 1 "+5V" H 10450 1240 50  0000 C CNN
 F 2 "" H 10450 1100 50  0001 C CNN
@@
 $EndComp
 $Comp
-L GND #PWR026
+L GND #PWR30
 U 1 1 5AA0C877
 P 10450 1550
-F 0 "#PWR026" H 10450 1300 50  0001 C CNN
+F 0 "#PWR30" H 10450 1300 50  0001 C CNN
 F 1 "GND" H 10450 1400 50  0000 C CNN
 F 2 "" H 10450 1550 50  0001 C CNN
@@
 Wire Wire Line
 	10450 1250 10450 1100
-$Comp
-L SW_DPST_x2 SW1
-U 1 1 5AA0D13D
-P 7550 2400
-F 0 "SW1" H 7550 2525 50  0000 C CNN
-F 1 "SW_DPST_x2" H 7550 2300 50  0000 C CNN
-F 2 "Buttons_Switches_SMD:SW_SPST_B3U-1000P" H 7550 2400 50  0001 C CNN
-F 3 "https://www.digikey.ca/product-detail/en/omron-electronics-inc-emc-div/B3U-1000P/SW1020CT-ND/1534357" H 7550 2400 50  0001 C CNN
-	1    7550 2400
-	1    0    0    -1
-$EndComp
 Wire Wire Line
 	7350 2400 7200 2400
 $Comp
-L GND #PWR027
+L GND #PWR27
 U 1 1 5AA0D26D
 P 7950 2500
-F 0 "#PWR027" H 7950 2250 50  0001 C CNN
+F 0 "#PWR27" H 7950 2250 50  0001 C CNN
 F 1 "GND" H 7950 2350 50  0000 C CNN
 F 2 "" H 7950 2500 50  0001 C CNN
@@
 Text GLabel 7200 2400 0    49   Input ~ 0
 RESET
-$Comp
-L SW_DPST_x2 SW1
-U 2 1 5AA0D563
-P 10050 2400
-F 0 "SW1" H 10050 2525 50  0000 C CNN
-F 1 "SW_DPST_x2" H 10050 2300 50  0000 C CNN
-F 2 "Buttons_Switches_SMD:SW_SPST_B3U-1000P" H 10050 2400 50  0001 C CNN
-F 3 "https://www.digikey.ca/product-detail/en/omron-electronics-inc-emc-div/B3U-1000P/SW1020CT-ND/1534357" H 10050 2400 50  0001 C CNN
-	2    10050 2400
-	1    0    0    -1
-$EndComp
 Wire Wire Line
 	9850 2400 9700 2400
 $Comp
-L GND #PWR028
+L GND #PWR31
 U 1 1 5AA0D56A
 P 10450 2500
-F 0 "#PWR028" H 10450 2250 50  0001 C CNN
+F 0 "#PWR31" H 10450 2250 50  0001 C CNN
 F 1 "GND" H 10450 2350 50  0000 C CNN
 F 2 "" H 10450 2500 50  0001 C CNN
@@
 	7650 4500 8050 4500
 $Comp
-L GND #PWR029
+L GND #PWR28
 U 1 1 5AA0DEF7
 P 8550 4650
-F 0 "#PWR029" H 8550 4400 50  0001 C CNN
+F 0 "#PWR28" H 8550 4400 50  0001 C CNN
 F 1 "GND" H 8550 4500 50  0000 C CNN
 F 2 "" H 8550 4650 50  0001 C CNN
@@
 $EndComp
 Wire Wire Line
-	8350 4500 8550 4500
+	8550 4500 8350 4500
 Wire Wire Line
 	8550 3700 8550 4650
@@
 F 0 "MK3" H 10500 4450 50  0000 C CNN
 F 1 "Mounting_Hole" H 10500 4375 50  0000 C CNN
-F 2 "" H 10500 4250 50  0001 C CNN
+F 2 "Mounting_Holes:MountingHole_3.2mm_M3" H 10500 4250 50  0001 C CNN
 F 3 "" H 10500 4250 50  0001 C CNN
 	1    10500 4250
@@
 F 0 "MK2" H 10000 4800 50  0000 C CNN
 F 1 "Mounting_Hole" H 10000 4725 50  0000 C CNN
-F 2 "" H 10000 4600 50  0001 C CNN
+F 2 "Mounting_Holes:MountingHole_3.2mm_M3" H 10000 4600 50  0001 C CNN
 F 3 "" H 10000 4600 50  0001 C CNN
 	1    10000 4600
@@
 L Mounting_Hole MK4
 U 1 1 5AED6AC9
-P 10600 4600
-F 0 "MK4" H 10600 4800 50  0000 C CNN
-F 1 "Mounting_Hole" H 10600 4725 50  0000 C CNN
-F 2 "" H 10600 4600 50  0001 C CNN
-F 3 "" H 10600 4600 50  0001 C CNN
-	1    10600 4600
+P 10500 4600
+F 0 "MK4" H 10500 4800 50  0000 C CNN
+F 1 "Mounting_Hole" H 10500 4725 50  0000 C CNN
+F 2 "Mounting_Holes:MountingHole_3.2mm_M3" H 10500 4600 50  0001 C CNN
+F 3 "" H 10500 4600 50  0001 C CNN
+	1    10500 4600
 	1    0    0    -1
 $EndComp
@@
 	1    0    0    -1
 $EndComp
+$Comp
+L SW_SPST SW1
+U 1 1 5AEEC585
+P 7550 2400
+F 0 "SW1" H 7550 2525 50  0000 C CNN
+F 1 "SW_SPST" H 7550 2300 50  0000 C CNN
+F 2 "Buttons_Switches_SMD:SW_SPST_B3U-1000P" H 7550 2400 50  0001 C CNN
+F 3 "https://www.digikey.ca/product-detail/en/omron-electronics-inc-emc-div/B3U-1000P/SW1020CT-ND/1534357" H 7550 2400 50  0001 C CNN
+	1    7550 2400
+	1    0    0    -1
+$EndComp
+$Comp
+L SW_SPST SW2
+U 1 1 5AEEC7E9
+P 10050 2400
+F 0 "SW2" H 10050 2525 50  0000 C CNN
+F 1 "SW_SPST" H 10050 2300 50  0000 C CNN
+F 2 "Buttons_Switches_SMD:SW_SPST_B3U-1000P" H 10050 2400 50  0001 C CNN
+F 3 "https://www.digikey.ca/product-detail/en/omron-electronics-inc-emc-div/B3U-1000P/SW1020CT-ND/1534357" H 10050 2400 50  0001 C CNN
+	1    10050 2400
+	1    0    0    -1
+$EndComp
+$Comp
+L R R28
+U 1 1 5AEF9229
+P 7300 2250
+F 0 "R28" V 7380 2250 50  0000 C CNN
+F 1 "10k" V 7300 2250 50  0000 C CNN
+F 2 "Resistors_SMD:R_0805" V 7230 2250 50  0001 C CNN
+F 3 "" H 7300 2250 50  0001 C CNN
+	1    7300 2250
+	-1   0    0    1
+$EndComp
+$Comp
+L +5V #PWR24
+U 1 1 5AEF9444
+P 7300 2100
+F 0 "#PWR24" H 7300 1950 50  0001 C CNN
+F 1 "+5V" H 7300 2240 50  0000 C CNN
+F 2 "" H 7300 2100 50  0001 C CNN
+F 3 "" H 7300 2100 50  0001 C CNN
+	1    7300 2100
+	1    0    0    -1
+$EndComp
+Connection ~ 7300 2400
+Text GLabel 9500 1350 0    49   Input ~ 0
+52(SCK)
+Text GLabel 10300 1350 2    49   Input ~ 0
+51(MOSI)
+Text GLabel 9500 1250 0    49   Input ~ 0
+50(MISO)
+Text GLabel 9700 2400 0    49   Input ~ 0
+37
+Text GLabel 7100 3700 0    49   Input ~ 0
+36
+Text GLabel 7100 4100 0    49   Input ~ 0
+35
+Text GLabel 7100 4500 0    49   Input ~ 0
+34
 $EndSCHEMATC
