File: KiCAD/OBC-PDB.kicad_pcb (KiCad board)
At the start: 2 copper layers, 127 parts, among them J1 Screw_Terminal_01x02, J10 Screw_Terminal_01x02, J11 Screw_Terminal_01x02, J12 Screw_Terminal_01x02, J13 Screw_Terminal_01x02, J14 Screw_Terminal_01x02, J15 Screw_Terminal_01x02, J16 Screw_Terminal_01x02, J17 Screw_Terminal_01x02, J19 Screw_Terminal_01x02, J2 Conn_02x03_Odd_Even, J20 Screw_Terminal_01x02, J21 Conn_01x01, J22 GS2, J23 uSD, J24 Conn_01x08, J25 Conn_01x16, J3 Screw_Terminal_01x02, J4 Screw_Terminal_01x02, J5 Screw_Terminal_01x02, J6 Screw_Terminal_01x02, J7 Screw_Terminal_01x02, J8 Screw_Terminal_01x02, J9 Screw_Terminal_01x02, SW1 SW_DPST_x2, U10 MAX6675, U11 MAX6675, U12 DS18B20, U13 DRV8825, U14 TCA9548A_TSSOP, U2 TPS565208, U3 ATMEGA2560-16AU, U4 Si8660, U6 MAX6675, U7 MAX6675, U8 DS1307Z+

Commit message: transfer for mechanical step
Parts:
- removed F1: 6.25, Fuse_Holders_and_Fuses:Fuseholder5x20_horiz_open_lateral_Type-II
- added C30: 10n, Capacitors_SMD:C_0805, F.Cu at (160.7, 66.4)
- added D7: D, Resistors_THT:R_Axial_DIN0204_L3.6mm_D1.6mm_P5.08mm_Horizontal, F.Cu at (62.0, 57.9)
- added J18: Conn_02x20_Top_Bottom, Pin_Headers:Pin_Header_Straight_2x20_Pitch2.54mm, F.Cu at (238.8, 61.6)
- added L2: 10uH, kicad-footprints:L-1008, F.Cu at (125.1, 101.0)
- added MK2: Mounting_Hole, Mounting_Holes:MountingHole_3.2mm_M3, F.Cu at (238.8, 51.4)
- added MK3: Mounting_Hole, Mounting_Holes:MountingHole_3.2mm_M3, F.Cu at (50.2, 140.3)
- added MK4: Mounting_Hole, Mounting_Holes:MountingHole_3.2mm_M3, F.Cu at (238.8, 140.3)
- added R28: 10k, Resistors_SMD:R_0805, F.Cu at (84.8, 80.7)
- added SW2: SW_SPST, Buttons_Switches_SMD:SW_SPST_B3U-1000P, F.Cu at (84.7, 90.2)
- added U1: LP2985-3.3, TO_SOT_Packages_SMD:SOT-23-5, F.Cu at (157.3, 63.8)
- added U5: PCA9306, Housings_SSOP:VSSOP-8_2.3x2mm_Pitch0.5mm, F.Cu at (92.0, 110.0)
- added U9: MPU-9250, Housings_DFN_QFN:QFN-24-1EP_3x3mm_Pitch0.4mm, F.Cu at (78.7, 104.1)
- added Y1: 16MHz, Crystals:Crystal_HC49-U_Vertical, F.Cu at (113.9, 79.4)
- added Y2: 32.768k, Crystals:Crystal_C26-LF_d2.1mm_l6.5mm_Horizontal, F.Cu at (182.9, 95.3)
- C1, C2: footprint Capacitors_SMD:C_1210 -> Capacitors_SMD:C_0805
- J22: moved to B.Cu
- SW1: value SW_DPST_x2 -> SW_SPST
- U13: footprint Housings_SSOP:HTSSOP-20-1EP_4.4x6.5mm_Pitch0.65mm_ThermalPad -> Housings_SSOP:HTSSOP-32_6.1x11mm_Pitch0.65mm_ThermalPad
- moved SPI3 203.6 mm to (228.0, 101.0)
- moved SPI1 195.3 mm to (215.3, 101.0)
- moved SPI2 192.3 mm to (221.6, 101.0)
- moved J19 180.1 mm to (204.5, 52.1)
- moved J7 169.9 mm to (193.0, 138.8), turned to 180 degrees
- moved J17 154.1 mm to (193.7, 52.1)
- moved LoRa1 152.5 mm to (204.5, 65.4), turned to 270 degrees
- moved J23 151.7 mm to (184.2, 72.4)
- moved J4 147.7 mm to (182.2, 138.8), turned to 180 degrees
- moved I2C3 139.9 mm to (225.4, 126.4)
- moved BT1 136.1 mm to (168.3, 81.8), turned to 90 degrees
- moved I2C2 131.7 mm to (219.7, 126.4)
- moved MK1 127.1 mm to (50.2, 51.4)
- moved U8 123.8 mm to (188.0, 97.2)
- moved I2C1 119.2 mm to (214.6, 126.4)
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Connections:
- C3 pad 1: Net-(C3-Pad1) -> +12V
- C4 pad 1: Net-(C3-Pad1) -> +12V
- D4 pad 2: Net-(D4-Pad2) -> 36
- D5 pad 2: Net-(D5-Pad2) -> 35
- D6 pad 2: Net-(D6-Pad2) -> 34
- Hall1 pad 2: Net-(Hall1-Pad2) -> -BATT
- J11 pad 1: Net-(J11-Pad1) -> 40
- J11 pad 2: Net-(J11-Pad2) -> 41
- J13 pad 1: Net-(J13-Pad1) -> 38
- J2 pad 1: MISO -> 50(MISO)
- J2 pad 3: SCK -> 52(SCK)
- J2 pad 4: MOSI -> 51(MOSI)
- J23 pad 2: Net-(J23-Pad2) -> 13(PWM)
- J23 pad 6: mcdigxxx -> 12(PWM)
- J25 pad 11: digipin -> 1(TX0)
- J25 pad 12: digipin -> 0(RX0)
- J25 pad 13: digipin -> 4(PWM)
- J25 pad 14: digipin -> A0
- J25 pad 4: digipin -> 3(PWM)
- J25 pad 6: digipin -> 2(PWM)
- J4 pad 1: Net-(J4-Pad1) -> A10
- J4 pad 2: Net-(J4-Pad2) -> A11
- J5 pad 1: Net-(J5-Pad1) -> 31
- J5 pad 2: Net-(J5-Pad2) -> 32
- J7 pad 1: Net-(J7-Pad1) -> A9
- J7 pad 2: Net-(J7-Pad2) -> -BATT
- J8 pad 1: Net-(J8-Pad1) -> 33
- LoRa1 pad 3: mcdigxxx -> Net-(LoRa1-Pad3)
- LoRa1 pad 4: mcdigxxx -> Net-(LoRa1-Pad4)
- LoRa1 pad 8: mcdigxxx -> Net-(LoRa1-Pad8)
- LoRa1 pad 9: mcdigxxx -> Net-(LoRa1-Pad9)
- R10 pad 2: Net-(Hall1-Pad2) -> Hall1
- R11 pad 2: -BATT -> Hall2
- R12 pad 2: -BATT -> Hall3
- R13 pad 2: -BATT -> Hall4
- R14 pad 2: -BATT -> Hall6
- R15 pad 2: -BATT -> Hall5
- R23 pad 2: mcdigxxx -> A8
- SPI1 pad 2: 53(SS) -> Net-(SPI1-Pad2)
- U10 pad 6: mcdigxxx -> 45(PWM)
- U11 pad 6: mcdigxxx -> 42
- U12 pad 2: mcdigxxx -> A8
- U13 pad 16: mcdigxxx -> 24
- U13 pad 20: mcdigxxx -> 25
- U13 pad 21: mcdigxxx -> 26
- U14 pad 1: Net-(U14-Pad1) -> 17(RX2)
- U14 pad 2: Net-(U14-Pad2) -> 16(TX2)
- U14 pad 21: Net-(U14-Pad21) -> 6(PWM)
- U2 pad 3: Net-(C3-Pad1) -> +12V
- U2 pad 5: Net-(C3-Pad1) -> +12V
- U4 pad 10: Net-(U4-Pad10) -> A12
- U4 pad 11: Net-(U4-Pad11) -> A13
- U4 pad 12: Net-(U4-Pad12) -> A14
- U4 pad 13: Net-(U4-Pad13) -> A15
- U4 pad 14: Net-(U4-Pad14) -> 22
- U4 pad 15: digiXX? -> 23
- U6 pad 6: mcdigxxx -> 43
- U7 pad 6: mcdigxxx -> 44(PWM)
Routing:
- net +5V: track 0.00 -> 958.1 mm, vias 0 -> 13
- net -BATT: track 0.00 -> 365.0 mm, vias 0 -> 59
- net 20(SDA): track 0.00 -> 217.2 mm, vias 0 -> 12
- net 21(SCL): track 0.00 -> 217.0 mm, vias 0 -> 13
- net 52(SCK): track 0.00 -> 212.9 mm, vias 0 -> 10
- net +12V: track 0.00 -> 212.4 mm, vias 0 -> 9
- net 50(MISO): track 0.00 -> 209.2 mm, vias 0 -> 7
- net +3V3: track 0.00 -> 206.3 mm, vias 0 -> 5
- net 51(MOSI): track 0.00 -> 155.7 mm, vias 0 -> 6
- net A0: track 0.00 -> 109.2 mm, vias 0 -> 4
- net A9: track 0.00 -> 108.2 mm, vias 0 -> 4
- net 3(PWM): track 0.00 -> 105.4 mm, vias 0 -> 4
- net 4(PWM): track 0.00 -> 104.5 mm, vias 0 -> 4
- net 0(RX0): track 0.00 -> 102.0 mm, vias 0 -> 4
- net 1(TX0): track 0.00 -> 100.9 mm, vias 0 -> 4
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- added copper zone on F.Cu, net +12V
- added copper zone on F.Cu, net +3V3
- added copper zone on F.Cu, net +5V
- added copper zone on B.Cu, net -BATT
- added copper zone on F.Cu, net -BATT
Other:
- board outline added: 200 x 100.3 mm
- board text added: "12V Supply Bus"
- board text added: "3V3 Supply Bus"
- board text added: "5V Supply Bus"
- board text added: "ATMEGA2560"
- board text added: "Analog In"
- board text added: "Buttons"
- board text added: "Gear Shift Select"
- board text added: "ICSP"
- board text added: "Memorial Baja"
- board text added: "Memorial Baja Electronic Instrumentation Cluster Version 1.0"
- board text added: "uSD"
